File: Eletrônica/MUDE - Rev B.brd (EAGLE design)
At the start: 27 x 18 mm, 31 parts, among them U2 Tiny85-20-SMT

Commit message: Rev A mostly finished
Parts:
- removed R2: (no value), wes:R0603
- removed SJ1: (no value), SparkFun-Passives:SJ_3
- removed T1, T2, T3, T4: (no value), zetex:SOT323
- removed TP4: TPSQTP14R, testpad:TP14R
- added CIN4: (no value), wes:C0805
- added J1, J2: 22-05-7038-03, con-molex:7395-03
- added Q1, Q2, Q3, Q4, Q5: MOSFET-NCHANNEL2N7002PW, SparkFun-DiscreteSemi:SOT323
- added R1, R3, R8: (no value), wes:R0603
- added RN2: (no value), resistor-dil:0603-ARV
- C5: device wes:C0603 -> wes:C0805
- U$3: value ISP_POGOISP_POGO -> ISP_POGOISP_LHOLE; device wes:ISP_POGO -> wes:ISP_POGO_LHOLE
- moved C9 9.55 mm to (17.5, 1.91)
- moved CIN3 9.44 mm to (6.03, 2.70), turned to 270 degrees
- moved C5 8.96 mm to (15.2, 2.06)
- moved C6 8.91 mm to (10.2, 2.54)
- moved CIN1 8.91 mm to (12.7, 5.87)
- moved U1 8.91 mm to (12.7, 2.54)
- moved RN1 8.47 mm to (21.0, 12.1), turned to 180 degrees
- moved CLOGIC 8.44 mm to (28.1, 2.70)
- moved C1 8.44 mm to (31.1, 2.70)
- moved C2 8.28 mm to (33.5, 6.35)
- moved C3 8.28 mm to (21.0, 9.84)
- moved C4 8.28 mm to (21.0, 2.86)
- moved C7 8.28 mm to (32.4, 11.6)
- moved CP 8.28 mm to (32.4, 10.0)
- moved R5 8.28 mm to (32.4, 13.2)
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Connections:
- removed net N$15: CIN3.1, FB.1
- removed net N$3: CIN1.1, CIN2.1, FB.2, U1.1, U1.3
- removed net N$8: R2.2, SJ1.2
- new net ATTINYOUT: J2.3, R3.1
- new net N$14: Q3.1, R1.2
- new net N$16: Q3.3, Q4.1, RN2.4
- new net N$18: Q5.3, R3.2, RN2.7
- new net N$21: Q4.3, R8.2, RN2.3
- new net NEOPIXELS: J1.3, R8.1
- new net V+: CIN1.1, CIN2.1, FB.2, RN2.2, RN2.5, RN2.6, U1.1, U1.3
- new net VIN: CIN3.1, CIN4.1, FB.1, J1.2, J2.2
- net +3V3: now also U$1.9; no longer SJ1.3
- net DATAOUT: now also R1.1
- net GND: now also CIN4.2, J1.1, J2.1, Q3.2, Q4.2, Q5.2; no longer SJ1.1
- net MISO: now also RN2.1
- net N$17: now also Q1.1, Q2.1; no longer T1.2, T4.2
- net N$2: now also Q5.1, RN2.8; no longer R2.1, U$1.9
- net N$7: now also Q2.3; no longer T4.1
- net N$9: now also Q1.3; no longer T1.1
- net SCL/SCK: now also Q1.2; no longer T1.3
- net SDA/MOSI: now also Q2.2; no longer T4.3
Routing:
- net V+: track 0.00 -> 22.1 mm, vias 0 -> 2
- net +3V3: track 35.0 -> 49.1 mm
- net MISO: track 5.33 -> 17.0 mm, vias 1 -> 3
- net DATAOUT: track 0.00 -> 9.65 mm, vias 0 -> 2
- net N$16: track 0.00 -> 9.59 mm
- net N$18: track 0.00 -> 8.27 mm
- net N$21: track 0.00 -> 7.86 mm
- net N$17: track 3.35 -> 10.3 mm, vias 0 -> 2
- net N$4: track 0.00 -> 5.37 mm
- net I2C-SWITCH: track 20.1 -> 15.4 mm
- net N$6: track 0.00 -> 3.89 mm
- net N$3: track 3.50 -> 0.00 mm
- net ATTINYOUT: track 0.00 -> 3.37 mm
- net N$9: track 8.38 -> 11.6 mm
- net N$14: track 0.00 -> 3.14 mm
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- added copper zone on layer 1, net N$5
- added copper zone on layer 1, net VIN
Other:
- board size 27 x 18 mm -> 35 x 16 mm
