File: Eletrônica/MUDE - Rev B.sch (EAGLE design)
At the start: 31 parts, among them U2 Tiny85-20-SMT

Commit message: Rev A mostly finished
Parts:
- removed R2: (no value), wes:R-EU_R0603
- removed SJ1: (no value), SparkFun-Passives:SOLDERJUMPER_2WAYS
- removed T1, T3, T4: (no value), zetex:NPNSOT323
- removed T2: (no value), zetex:PNPSOT323
- removed TP4: TPSQTP14R, testpad:TPSQTP14R
- added CIN4: (no value), wes:C-EUC0805
- added J1, J2: 22-05-7038-03, con-molex:22-05-7038-03
- added Q1, Q2, Q3, Q4, Q5: MOSFET-NCHANNEL2N7002PW, SparkFun-DiscreteSemi:MOSFET-NCHANNEL2N7002PW
- added R1, R3, R8: (no value), wes:R-EU_R0603
- added RN2: (no value), resistor-dil:4R-N0603-ARV
- C5: device wes:C-EUC0603 -> wes:C-EUC0805
- U$3: value ISP_POGOISP_POGO -> ISP_POGOISP_LHOLE; device wes:ISP_POGOISP_POGO -> wes:ISP_POGOISP_LHOLE
Connections:
- removed net N$15: CIN3.1, FB.1
- removed net N$3: CIN1.1, CIN2.1, FB.2, U1.EN, U1.IN
- removed net N$8: R2.2, SJ1.2
- new net ATTINYOUT: J2-3.S, R3.1
- new net N$14: Q3.G, R1.2
- new net N$16: Q3.D, Q4.G, RN2D.1
- new net N$18: Q5.D, R3.2, RN2B.2
- new net N$21: Q4.D, R8.2, RN2C.1
- new net NEOPIXELS: J1-3.S, R8.1
- new net V+: CIN1.1, CIN2.1, FB.2, RN2B.1, RN2C.2, RN2D.2, U1.EN, U1.IN
- new net VIN: CIN3.1, CIN4.1, FB.1, J1-2.S, J2-2.S
- net +3V3: now also U$1.AD0; no longer SJ1.3
- net DATAOUT: now also R1.1
- net GND: now also CIN4.2, J1-1.S, J2-1.S, Q3.S, Q4.S, Q5.S; no longer SJ1.1
- net MISO: now also RN2A.1
- net N$17: now also Q1.G, Q2.G; no longer T1.B, T4.B
- net N$2: now also Q5.G, RN2A.2; no longer R2.1, U$1.AD0
- net N$7: now also Q2.D; no longer T4.C
- net N$9: now also Q1.D; no longer T1.C
- net SCL/SCK: now also Q1.S; no longer T1.E
- net SDA/MOSI: now also Q2.S; no longer T4.E
